Commit message: feat: adding interlagos camera world

File: code/src/lia_robot/description/camera.xacro (robot description, xacro)
@@ -4,5 +4,5 @@
         <parent link="chassis"/>
         <child link="camera_link"/>
-        <origin xyz="0.13 0 0.02" rpy="0 ${-pi/9} 0"/>
+        <origin xyz="0.13 0 0.10" rpy="0 ${pi/12} 0"/>
     </joint>
     <link name="camera_link">

Commit message: feat: updating robot chassis

File: code/src/lia_robot/description/camera.xacro (robot description, xacro)
@@ -4,10 +4,11 @@
         <parent link="chassis"/>
         <child link="camera_link"/>
-        <origin xyz="0.13 0 0.10" rpy="0 ${pi/12} 0"/>
+        <!-- <origin xyz="0.13 0 0.10" rpy="0 ${pi/12} 0"/> -->
+        <origin xyz="0.095 0 0.11" rpy="0 0 0"/>
     </joint>
     <link name="camera_link">
         <visual>
             <geometry>
-                <box size="0.001 0.10 0.03"/>
+                <!-- <box size="0.001 0.10 0.03"/> -->
             </geometry>
             <material name="red"/>
@@ -27,5 +28,6 @@
             <update_rate>10</update_rate>
             <camera>
-                <horizontal_fov>1.089</horizontal_fov>
+                <!-- <horizontal_fov>1.089</horizontal_fov> -->
+                <horizontal_fov>0.7835</horizontal_fov>
                 <image>
                     <format>R8G8B8</format>

File: code/src/lia_robot/description/robot_core.xacro (robot description, xacro)
@@ -17,4 +17,7 @@
         <color rgba="1 1 0 1"/>
     </material>
+    <material name="deeporange" >
+        <color rgba="0.8627450980392157 0.30196078431372547 0.00392156862745098 1.0" />
+    </material>
     <!-- BASE LINK -->
     <link name="base_link">
@@ -33,15 +36,15 @@
             <!-- adding lia mesh -->
             <geometry>
-                <mesh filename="file://$(find lia_robot)/meshes/lia_chassis.stl"/>
-                <box size="0.22 0.10 0.05"/>
+                <mesh filename="file://$(find lia_robot)/meshes/lia_car_chassis_v2.stl"/>
+                <!-- <box size="0.22 0.10 0.05"/> -->
             </geometry>
-            <material name="yellow"/>
+            <material name="orange"/>
         </visual>
         <collision>
             <!-- <origin xyz="0.075 0 0"/> -->
-            <origin xyz="0.14 0 0.018"/>
+            <origin xyz="0.116 0 0.018"/>
             <geometry>
-                <box size="0.22 0.10 0.05"/>
-                <!-- <mesh filename="package://lia_robot/meshes/lia_chassis.stl"/> -->
+                <box size="0.17 0.106 0.05"/>
+                <!-- <mesh filename="package://lia_robot/meshes/lia_car_chassis_v2.stl"/> -->
             </geometry>
         </collision>
@@ -51,5 +54,6 @@
     </link>
     <gazebo reference="chassis">
-        <material>Gazebo/DarkYellow</material>
+        <!-- <material>Gazebo/DarkYellow</material> -->
+        <material>deeporange</material>
     </gazebo>
     <!-- LEFT WHEEL LINK -->
@@ -57,5 +61,5 @@
         <parent link="base_link"/>
         <child link="left_wheel"/>
-        <origin xyz="0 0.07 0" rpy="-${pi/2} 0 0" />
+        <origin xyz="0 0.045 0" rpy="-${pi/2} 0 0" />
         <axis xyz="0 0 1"/>
     </joint>
@@ -83,5 +87,5 @@
         <parent link="base_link"/>
         <child link="right_wheel"/>
-        <origin xyz="0 -0.07 0" rpy="${pi/2} 0 0" />
+        <origin xyz="0 -0.045 0" rpy="${pi/2} 0 0" />
         <axis xyz="0 0 -1"/>
     </joint>
@@ -109,5 +113,5 @@
         <parent link="chassis"/>
         <child link="caster_wheel"/>
-        <origin xyz="0.151 0 -0.0075"/>
+        <origin xyz="0.165 0.028 -0.0075"/>
     </joint>
     <link name="caster_wheel">
@@ -136,5 +140,5 @@
         <parent link="chassis"/>
         <child link="caster_wheel2"/>
-        <origin xyz="0.205 0 -0.0075"/>
+        <origin xyz="0.165 -0.028 -0.0075"/>
     </joint>
     <link name="caster_wheel2">

Commit message: feat: vision improvements

File: code/src/lia_robot/description/camera.xacro (robot description, xacro)
@@ -5,5 +5,5 @@
         <child link="camera_link"/>
         <!-- <origin xyz="0.13 0 0.10" rpy="0 ${pi/12} 0"/> -->
-        <origin xyz="0.095 0 0.11" rpy="0 0 0"/>
+        <origin xyz="0.095 0 0.12" rpy="0 ${pi/12} 0"/>
     </joint>
     <link name="camera_link">

File: code/src/lia_robot/description/robot_core.xacro (robot description, xacro)
@@ -54,6 +54,6 @@
     </link>
     <gazebo reference="chassis">
-        <!-- <material>Gazebo/DarkYellow</material> -->
-        <material>deeporange</material>
+        <material>Gazebo/DarkYellow</material>
+        <!-- <material>Gazebo/deeporange</material> -->
     </gazebo>
     <!-- LEFT WHEEL LINK -->
