Commit message: feat: finishing LIA urdf

File: code/src/lia_robot/description/robot_core.xacro (robot description, xacro)
@@ -28,11 +28,4 @@
     </joint>
     <link name="chassis">
-        <!-- <visual>
-            <origin xyz="0.09 0 0.05"/>
-            <geometry>
-                <box size="0.18 0.10 0.10"/>
-            </geometry>
-            <material name="yellow"/>
-        </visual> -->
         <visual>
             <origin xyz="0.075 0 0"/>
@@ -44,11 +37,11 @@
         </visual>
         <collision>
-            <origin xyz="0.15 0 0.075"/>
+            <origin xyz="0.075 0 0"/>
             <geometry>
-                <box size="0.3 0.3 0.15"/>
+                <mesh filename="package://lia_robot/meshes/lia_chassis.stl"/>
             </geometry>
         </collision>
-        <xacro:inertial_box mass="0.5" x="0.3" y="0.3" z="0.15">
-            <origin xyz="0.15 0 0.075" rpy="0 0 0"/>
+        <xacro:inertial_box mass="0.5" x="0.18" y="0.10" z="0.10">
+            <origin xyz="0 0 0" rpy="0 0 0"/>
         </xacro:inertial_box>
     </link>
@@ -69,8 +62,8 @@
         <collision>
             <geometry>
-                <cylinder radius="0.025" length="0.05"/>
+                <cylinder radius="0.025" length="0.01"/>
             </geometry>
         </collision>
-        <xacro:inertial_cylinder mass="0.1" length="0.05" radius="0.025">
+        <xacro:inertial_cylinder mass="0.1" length="0.01" radius="0.025">
             <origin xyz="0 0 0" rpy="0 0 0"/>
         </xacro:inertial_cylinder>
@@ -92,12 +85,12 @@
         <collision>
             <geometry>
-                <cylinder radius="0.025" length="0.05"/>
+                <cylinder radius="0.025" length="0.01"/>
             </geometry>
         </collision>
-        <xacro:inertial_cylinder mass="0.1" length="0.05" radius="0.025">
+        <xacro:inertial_cylinder mass="0.1" length="0.01" radius="0.025">
             <origin xyz="0 0 0" rpy="0 0 0"/>
         </xacro:inertial_cylinder>
     </link>
-    <!-- CASTER WHEEL LINK -->
+    <!-- FIRST CASTER WHEEL LINK -->
     <joint name="caster_wheel_joint" type="fixed">
         <parent link="chassis"/>
@@ -114,8 +107,30 @@
         <collision>
             <geometry>
-                <sphere radius="0.01"/>
+                <sphere radius="0.005"/>
             </geometry>
         </collision>
-        <xacro:inertial_sphere mass="0.1" radius="0.01">
+        <xacro:inertial_sphere mass="0.1" radius="0.005">
+            <origin xyz="0 0 0" rpy="0 0 0"/>
+        </xacro:inertial_sphere>
+    </link>
+    <!-- SECOND CASTER WHEEL LINK -->
+    <joint name="caster_wheel_joint2" type="fixed">
+        <parent link="chassis"/>
+        <child link="caster_wheel2"/>
+        <origin xyz="0.205 0 -0.0075"/>
+    </joint>
+    <link name="caster_wheel2">
+        <visual>
+            <geometry>
+                <sphere radius="0.005"/>
+            </geometry>
+            <material name="white"/>
+        </visual>
+        <collision>
+            <geometry>
+                <sphere radius="0.005"/>
+            </geometry>
+        </collision>
+        <xacro:inertial_sphere mass="0.1" radius="0.005">
             <origin xyz="0 0 0" rpy="0 0 0"/>
         </xacro:inertial_sphere>

Commit message: adding simulation files and tcc point

File: code/src/lia_robot/description/robot_core.xacro (robot description, xacro)
@@ -6,5 +6,5 @@
     </material>
     <material name="orange">
-        <color rgba="1 0.3 0.1 1"/>
+        <color rgba="${255/255} ${108/255} ${10/255} 1.0"/>
     </material>
     <material name="blue">
@@ -38,4 +38,5 @@
                 <mesh filename="file://$(find lia_robot)/meshes/lia_car_chassis_v2.stl"/>
                 <!-- <box size="0.22 0.10 0.05"/> -->
+                <!-- <mesh filename="package://lia_robot/meshes/lia_car_chassis_v2.stl"/> -->
             </geometry>
             <material name="orange"/>
@@ -54,5 +55,5 @@
     </link>
     <gazebo reference="chassis">
-        <material>Gazebo/DarkYellow</material>
+        <material>Gazebo/Orange</material>
         <!-- <material>Gazebo/deeporange</material> -->
     </gazebo>
@@ -69,5 +70,5 @@
                 <cylinder radius="0.025" length="0.01"/>
             </geometry>
-            <material name="black"/>
+            <material name="white"/>
         </visual>
         <collision>
@@ -81,5 +82,5 @@
     </link>
     <gazebo reference="left_wheel">
-        <material>Gazebo/Black</material>
+        <material>Gazebo/White</material>
     </gazebo>
     <!-- RIGHT WHEEL LINK -->
@@ -95,5 +96,5 @@
                 <cylinder radius="0.025" length="0.01"/>
             </geometry>
-            <material name="black"/>
+            <material name="white"/>
         </visual>
         <collision>
@@ -107,5 +108,5 @@
     </link>
    <gazebo reference="right_wheel">
-        <material>Gazebo/Black</material>
+        <material>Gazebo/White</material>
     </gazebo>
     <!-- FIRST CASTER WHEEL LINK -->
@@ -163,3 +164,12 @@
         <mu2 value="0.001" />
     </gazebo>
+    <gazebo>
+        <plugin filename="libgazebo_ros_p3d.so" name="lia_groundtruth_sim">
+        <update_rate>100.0</update_rate>
+        <body_name>base_link</body_name>
+        <topic_name>ground_truth/state</topic_name>
+        <gaussian_noise>0.0</gaussian_noise>
+        <frame_name>map</frame_name>
+      </plugin>
+    </gazebo>
 </robot>
